File: kicad_project/usb_hub.kicad_sch (KiCad schematic)
At the start: 52 parts, among them J1 USB4105-GF-A, J2 UJ2-ADH-3-TH, U2 CY7C65632-48AXCT, U3 USBLC6-2SC6, U4 USBLC6-2SC6, U5 USBLC6-2SC6, U6 BD2221G-LBTR, U7 BD2221G-LBTR

Commit message: Fill in all part numbers, add pcbinv bom job
Parts:
- FB1, FB2, FB4, FB5: LibRef (none) -> 742792121
- R1: LibRef (none) -> ERJ-8ENF1003V; SKU (none) -> P100KFCT-ND
- R1: LibRef (none) -> ERJ-8ENF2700V; SKU (none) -> P270FCT-ND
- R1: LibRef (none) -> RC1206FR-075K1L; SKU (none) -> 311-5.10KFRCT-ND
- R1: LibRef (none) -> P300FCT-ND; SKU (none) -> P300FCT-ND
- R1: LibRef (none) -> ERJ-8ENF1002V; SKU (none) -> P10.0KFCT-ND
- R1: LibRef (none) -> RC1206FR-07649RL; SKU (none) -> 311-649FRCT-ND
- R1: LibRef (none) -> ERJ-8ENF4702V; SKU (none) -> P47.0KFCT-ND
Changed lines of the file:
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@@
       (effects (font (size 1.27 1.27)) hide)
     )
+    (property "Description" "CAP CER 2.2uF 50V X7R 1206" (at 218.44 97.79 0)
+      (effects (font (size 1.27 1.27)) hide)
+    )
     (pin "1")
     (pin "2")
@@
       (effects (font (size 1.27 1.27)) hide)
     )
-    (property "LibRef" "" (at 241.3 219.71 0)
+    (property "LibRef" "ERJ-8ENF1003V" (at 241.3 219.71 0)
+      (effects (font (size 1.27 1.27)) hide)
+    )
+    (property "SKU" "P100KFCT-ND" (at 241.3 219.71 0)
       (effects (font (size 1.27 1.27)) hide)
     )
@@
       (effects (font (size 1.27 1.27)) hide)
     )
-    (property "LibRef" "" (at 302.26 223.52 0)
+    (property "LibRef" "ERJ-8ENF2700V" (at 302.26 223.52 0)
+      (effects (font (size 1.27 1.27)) hide)
+    )
+    (property "Description" "RES SMD 270 Ohm 1% 1/4W 1206" (at 302.26 223.52 0)
+      (effects (font (size 1.27 1.27)) hide)
+    )
+    (property "SKU" "P270FCT-ND" (at 302.26 223.52 0)
       (effects (font (size 1.27 1.27)) hide)
     )
@@
       (effects (font (size 1.27 1.27)) hide)
     )
-    (property "LibRef" "" (at 205.74 60.96 0)
+    (property "LibRef" "ERJ-8ENF1003V" (at 205.74 60.96 0)
+      (effects (font (size 1.27 1.27)) hide)
+    )
+    (property "SKU" "P100KFCT-ND" (at 205.74 60.96 0)
       (effects (font (size 1.27 1.27)) hide)
     )
@@
       (effects (font (size 1.27 1.27)) hide)
     )
-    (property "LibRef" "" (at 351.79 49.53 0)
+    (property "LibRef" "RC1206FR-075K1L" (at 351.79 49.53 0)
+      (effects (font (size 1.27 1.27)) hide)
+    )
+    (property "Description" "RES 5.1k Ohm 1% 1/4W 1206" (at 351.79 49.53 0)
+      (effects (font (size 1.27 1.27)) hide)
+    )
+    (property "SKU" "311-5.10KFRCT-ND" (at 351.79 49.53 0)
       (effects (font (size 1.27 1.27)) hide)
     )
@@
       (effects (font (size 1.27 1.27)) hide)
     )
-    (property "LibRef" "" (at 351.79 223.52 0)
+    (property "LibRef" "P300FCT-ND" (at 351.79 223.52 0)
+      (effects (font (size 1.27 1.27)) hide)
+    )
+    (property "Description" "RES SMD 300 Ohm 1% 1/4W 1206" (at 351.79 223.52 0)
+      (effects (font (size 1.27 1.27)) hide)
+    )
+    (property "SKU" "P300FCT-ND" (at 351.79 223.52 0)
       (effects (font (size 1.27 1.27)) hide)
     )
@@
       (effects (font (size 1.27 1.27)) hide)
     )
+    (property "Description" "CAP ALUM POLY 100uF 20% 35V T/H" (at 232.41 52.07 0)
+      (effects (font (size 1.27 1.27)) hide)
+    )
     (pin "1")
     (pin "2")
@@
       (effects (font (size 1.27 1.27)) hide)
     )
-    (property "LibRef" "" (at 90.17 125.73 0)
+    (property "LibRef" "ERJ-8ENF1002V" (at 90.17 125.73 0)
+      (effects (font (size 1.27 1.27)) hide)
+    )
+    (property "SKU" "P10.0KFCT-ND" (at 90.17 125.73 0)
       (effects (font (size 1.27 1.27)) hide)
     )
@@
       (effects (font (size 1.27 1.27)) hide)
     )
-    (property "LibRef" "" (at 318.77 223.52 0)
+    (property "LibRef" "P300FCT-ND" (at 318.77 223.52 0)
+      (effects (font (size 1.27 1.27)) hide)
+    )
+    (property "Description" "RES SMD 300 Ohm 1% 1/4W 1206" (at 318.77 223.52 0)
+      (effects (font (size 1.27 1.27)) hide)
+    )
+    (property "SKU" "P300FCT-ND" (at 318.77 223.52 0)
       (effects (font (size 1.27 1.27)) hide)
     )
@@
       (effects (font (size 1.27 1.27)) hide)
     )
+    (property "Description" "CAP CER 2.2uF 50V X7R 1206" (at 218.44 52.07 0)
+      (effects (font (size 1.27 1.27)) hide)
+    )
     (pin "1")
     (pin "2")
@@
       (effects (font (size 1.27 1.27)) hide)
     )
-    (property "LibRef" "" (at 68.58 236.22 0)
+    (property "LibRef" "P300FCT-ND" (at 68.58 236.22 0)
+      (effects (font (size 1.27 1.27)) hide)
+    )
+    (property "Description" "RES SMD 300 Ohm 1% 1/4W 1206" (at 68.58 236.22 0)
+      (effects (font (size 1.27 1.27)) hide)
+    )
+    (property "SKU" "P300FCT-ND" (at 68.58 236.22 0)
       (effects (font (size 1.27 1.27)) hide)
     )
@@
       (effects (font (size 1.27 1.27)) hide)
     )
-    (property "LibRef" "" (at 226.06 46.99 0)
+    (property "LibRef" "742792121" (at 226.06 46.99 0)
+      (effects (font (size 1.27 1.27)) hide)
+    )
+    (property "Description" "FERRITE BEAD 300 OHM 1206 1LN" (at 226.06 46.99 0)
       (effects (font (size 1.27 1.27)) hide)
     )
@@
       (effects (font (size 1.27 1.27)) hide)
     )
+    (property "Description" "CAP ALUM POLY 100uF 20% 35V T/H" (at 233.68 97.79 0)
+      (effects (font (size 1.27 1.27)) hide)
+    )
     (pin "1")
     (pin "2")
@@
       (effects (font (size 1.27 1.27)) hide)
     )
-    (property "LibRef" "" (at 213.36 247.65 0)
+    (property "LibRef" "ERJ-8ENF1003V" (at 213.36 247.65 0)
+      (effects (font (size 1.27 1.27)) hide)
+    )
+    (property "SKU" "P100KFCT-ND" (at 213.36 247.65 0)
       (effects (font (size 1.27 1.27)) hide)
     )
@@
       (effects (font (size 1.27 1.27)) hide)
     )
-    (property "LibRef" "" (at 212.09 214.63 0)
+    (property "LibRef" "ERJ-8ENF1003V" (at 212.09 214.63 0)
+      (effects (font (size 1.27 1.27)) hide)
+    )
+    (property "SKU" "P100KFCT-ND" (at 212.09 214.63 0)
       (effects (font (size 1.27 1.27)) hide)
     )
@@
       (effects (font (size 1.27 1.27)) hide)
     )
-    (property "LibRef" "" (at 58.42 43.18 0)
+    (property "LibRef" "742792121" (at 58.42 43.18 0)
+      (effects (font (size 1.27 1.27)) hide)
+    )
+    (property "Description" "FERRITE BEAD 300 OHM 1206 1LN" (at 58.42 43.18 0)
       (effects (font (size 1.27 1.27)) hide)
     )
@@
       (effects (font (size 1.27 1.27)) hide)
     )
-    (property "LibRef" "" (at 83.82 120.65 0)
+    (property "LibRef" "RC1206FR-07649RL" (at 83.82 120.65 0)
+      (effects (font (size 1.27 1.27)) hide)
+    )
+    (property "Description" "RES 649 Ohm 1% 1/4W 1206" (at 83.82 120.65 0)
+      (effects (font (size 1.27 1.27)) hide)
+    )
+    (property "SKU" "311-649FRCT-ND" (at 83.82 120.65 0)
       (effects (font (size 1.27 1.27)) hide)
     )
@@
       (effects (font (size 1.27 1.27)) hide)
     )
-    (property "LibRef" "" (at 205.74 106.68 0)
+    (property "LibRef" "ERJ-8ENF1003V" (at 205.74 106.68 0)
+      (effects (font (size 1.27 1.27)) hide)
+    )
+    (property "SKU" "P100KFCT-ND" (at 205.74 106.68 0)
       (effects (font (size 1.27 1.27)) hide)
     )
@@
       (effects (font (size 1.27 1.27)) hide)
     )
-    (property "LibRef" "" (at 351.79 46.99 0)
+    (property "LibRef" "RC1206FR-075K1L" (at 351.79 46.99 0)
+      (effects (font (size 1.27 1.27)) hide)
+    )
+    (property "Description" "RES 5.1k Ohm 1% 1/4W 1206" (at 351.79 46.99 0)
+      (effects (font (size 1.27 1.27)) hide)
+    )
+    (property "SKU" "311-5.10KFRCT-ND" (at 351.79 46.99 0)
       (effects (font (size 1.27 1.27)) hide)
     )
@@
       (effects (font (size 1.27 1.27)) hide)
     )
-    (property "LibRef" "" (at 78.74 231.14 0)
+    (property "LibRef" "ERJ-8ENF1003V" (at 78.74 231.14 0)
+      (effects (font (size 1.27 1.27)) hide)
+    )
+    (property "SKU" "P100KFCT-ND" (at 78.74 231.14 0)
       (effects (font (size 1.27 1.27)) hide)
     )
@@
       (effects (font (size 1.27 1.27)) hide)
     )
-    (property "LibRef" "" (at 24.13 121.92 0)
+    (property "LibRef" "ERJ-8ENF1002V" (at 24.13 121.92 0)
+      (effects (font (size 1.27 1.27)) hide)
+    )
+    (property "SKU" "P10.0KFCT-ND" (at 24.13 121.92 0)
       (effects (font (size 1.27 1.27)) hide)
     )
@@
       (effects (font (size 1.27 1.27)) hide)
     )
-    (property "LibRef" "" (at 218.44 241.3 0)
+    (property "LibRef" "ERJ-8ENF1003V" (at 218.44 241.3 0)
+      (effects (font (size 1.27 1.27)) hide)
+    )
+    (property "SKU" "P100KFCT-ND" (at 218.44 241.3 0)
       (effects (font (size 1.27 1.27)) hide)
     )
@@
       (effects (font (size 1.27 1.27)) hide)
     )
-    (property "LibRef" "" (at 226.06 92.71 0)
+    (property "LibRef" "742792121" (at 226.06 92.71 0)
+      (effects (font (size 1.27 1.27)) hide)
+    )
+    (property "Description" "FERRITE BEAD 300 OHM 1206 1LN" (at 226.06 92.71 0)
       (effects (font (size 1.27 1.27)) hide)
     )
@@
       (effects (font (size 1.27 1.27)) hide)
     )
-    (property "LibRef" "" (at 217.17 208.28 0)
+    (property "LibRef" "ERJ-8ENF1003V" (at 217.17 208.28 0)
+      (effects (font (size 1.27 1.27)) hide)
+    )
+    (property "SKU" "P100KFCT-ND" (at 217.17 208.28 0)
       (effects (font (size 1.27 1.27)) hide)
     )
@@
       (effects (font (size 1.27 1.27)) hide)
     )
-    (property "LibRef" "" (at 29.21 137.16 0)
+    (property "LibRef" "ERJ-8ENF4702V" (at 29.21 137.16 0)
+      (effects (font (size 1.27 1.27)) hide)
+    )
+    (property "SKU" "P47.0KFCT-ND" (at 29.21 137.16 0)
       (effects (font (size 1.27 1.27)) hide)
     )
@@
       (effects (font (size 1.27 1.27)) hide)
     )
-    (property "LibRef" "" (at 335.28 223.52 0)
+    (property "LibRef" "ERJ-8ENF2700V" (at 335.28 223.52 0)
+      (effects (font (size 1.27 1.27)) hide)
+    )
+    (property "Description" "RES SMD 270 Ohm 1% 1/4W 1206" (at 335.28 223.52 0)
+      (effects (font (size 1.27 1.27)) hide)
+    )
+    (property "SKU" "P270FCT-ND" (at 335.28 223.52 0)
       (effects (font (size 1.27 1.27)) hide)
     )
@@
       (effects (font (size 1.27 1.27)) hide)
     )
-    (property "LibRef" "" (at 50.8 68.58 0)
+    (property "LibRef" "742792121" (at 50.8 68.58 0)
+      (effects (font (size 1.27 1.27)) hide)
+    )
+    (property "Description" "FERRITE BEAD 300 OHM 1206 1LN" (at 50.8 68.58 0)
       (effects (font (size 1.27 1.27)) hide)
     )
