File: kicad_project/usb_hub.kicad_sch (KiCad schematic)
At the start: 55 parts, among them J1 USB4105-GF-A, J2 UJ2-ADH-3-TH, U2 CY7C65632-48AXCT, U3 USBLC6-2SC6, U4 USBLC6-2SC6, U5 USBLC6-2SC6, U6 BD2221G-LBTR, U7 BD2221G-LBTR

Commit message: Finish schematic and placement for all remaining RP2354 power passives
Connections:
- net GND: now also J2.SH (Shield); no longer J2.9 (Shield)
Changed lines of the file:
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@@
 		(pin "B9"
 		)
-		(pin "S1"
+		(pin "SH"
 		)
 		(instances
@@
 		(pin "8"
 		)
-		(pin "9"
+		(pin "SH"
 		)
 		(instances
