File: kicad_project/PowerUSBPort.kicad_sch (KiCad schematic)
At the start: 10 parts, among them J1 USB4105-GF-A, U3 USBLC6-2SC6, U9 LD1117S33TR_SOT223

Commit message: Add part numbers for capacitors, start working on BoM job
Parts:
- C12: LibRef (none) -> CL31B106KLHNNNE; Supplier (none) -> Digi-Key
- C12: value 100n -> 100nF; LibRef (none) -> GRM319R72A104KA01D; Supplier (none) -> Digi-Key
- C12, C13: value 2.2u -> 2.2uF; LibRef (none) -> CL31B225KBHNNNE; SKU (none) -> 1276-1291-1-ND; Supplier (none) -> Digi-Key
- FB4, J1, R11, R12, U3, U9: Supplier (none) -> Digi-Key
Changed lines of the file:
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@@
       (effects (font (size 1.27 1.27)) (justify right))
     )
-    (property "Value" "2.2u" (at 128.27 80.0036 0)
+    (property "Value" "2.2uF" (at 128.27 80.0036 0)
       (effects (font (size 1.27 1.27)) (justify right))
     )
@@
       (effects (font (size 1.27 1.27)) hide)
     )
+    (property "Supplier" "Digi-Key" (at 125.73 78.74 0)
+      (effects (font (size 1.27 1.27)) hide)
+    )
+    (property "LibRef" "CL31B225KBHNNNE" (at 125.73 78.74 0)
+      (effects (font (size 1.27 1.27)) hide)
+    )
+    (property "SKU" "1276-1291-1-ND" (at 125.73 78.74 0)
+      (effects (font (size 1.27 1.27)) hide)
+    )
     (pin "1")
     (pin "2")
@@
     )
     (property "Datasheet" "~" (at 193.04 78.74 0)
+      (effects (font (size 1.27 1.27)) hide)
+    )
+    (property "Supplier" "Digi-Key" (at 193.04 78.74 0)
+      (effects (font (size 1.27 1.27)) hide)
+    )
+    (property "LibRef" "CL31B106KLHNNNE" (at 193.04 78.74 0)
       (effects (font (size 1.27 1.27)) hide)
     )
@@
       (effects (font (size 1.27 1.27)) hide)
     )
+    (property "Supplier" "Digi-Key" (at 121.92 101.6 0)
+      (effects (font (size 1.27 1.27)) hide)
+    )
+    (property "LibRef" "" (at 121.92 101.6 0)
+      (effects (font (size 1.27 1.27)) hide)
+    )
     (pin "1")
     (pin "2")
@@
       (effects (font (size 1.27 1.27)) hide)
     )
+    (property "Supplier" "Digi-Key" (at 111.76 82.55 0)
+      (effects (font (size 1.27 1.27)) hide)
+    )
+    (property "LibRef" "" (at 111.76 82.55 0)
+      (effects (font (size 1.27 1.27)) hide)
+    )
     (pin "1")
     (pin "2")
@@
       (effects (font (size 1.27 1.27)) (justify right))
     )
-    (property "Value" "100n" (at 163.83 80.0036 0)
+    (property "Value" "100nF" (at 163.83 80.0036 0)
       (effects (font (size 1.27 1.27)) (justify right))
     )
@@
       (effects (font (size 1.27 1.27)) hide)
     )
+    (property "SKU" "" (at 161.29 78.74 0)
+      (effects (font (size 1.27 1.27)) hide)
+    )
+    (property "Supplier" "Digi-Key" (at 161.29 78.74 0)
+      (effects (font (size 1.27 1.27)) hide)
+    )
+    (property "LibRef" "GRM319R72A104KA01D" (at 161.29 78.74 0)
+      (effects (font (size 1.27 1.27)) hide)
+    )
     (pin "1")
     (pin "2")
@@
       (effects (font (size 1.27 1.27)) (justify right))
     )
-    (property "Value" "2.2u" (at 146.05 80.0036 0)
+    (property "Value" "2.2uF" (at 146.05 80.0036 0)
       (effects (font (size 1.27 1.27)) (justify right))
     )
@@
     )
     (property "Datasheet" "~" (at 143.51 78.74 0)
+      (effects (font (size 1.27 1.27)) hide)
+    )
+    (property "Supplier" "Digi-Key" (at 143.51 78.74 0)
+      (effects (font (size 1.27 1.27)) hide)
+    )
+    (property "LibRef" "CL31B225KBHNNNE" (at 143.51 78.74 0)
+      (effects (font (size 1.27 1.27)) hide)
+    )
+    (property "SKU" "1276-1291-1-ND" (at 143.51 78.74 0)
       (effects (font (size 1.27 1.27)) hide)
     )
@@
       (effects (font (size 1.27 1.27)) hide)
     )
+    (property "Supplier" "Digi-Key" (at 111.76 80.01 0)
+      (effects (font (size 1.27 1.27)) hide)
+    )
+    (property "LibRef" "" (at 111.76 80.01 0)
+      (effects (font (size 1.27 1.27)) hide)
+    )
     (pin "1")
     (pin "2")
@@
     )
     (property "Datasheet" "http://www.st.com/st-web-ui/static/active/en/resource/technical/document/datasheet/CD00000544.pdf" (at 180.34 81.28 0)
+      (effects (font (size 1.27 1.27)) hide)
+    )
+    (property "Supplier" "Digi-Key" (at 177.8 74.93 0)
+      (effects (font (size 1.27 1.27)) hide)
+    )
+    (property "LibRef" "" (at 177.8 74.93 0)
       (effects (font (size 1.27 1.27)) hide)
     )
@@
       (effects (font (size 1.27 1.27)) hide)
     )
+    (property "Supplier" "Digi-Key" (at 135.89 74.93 0)
+      (effects (font (size 1.27 1.27)) hide)
+    )
+    (property "LibRef" "" (at 135.89 74.93 0)
+      (effects (font (size 1.27 1.27)) hide)
+    )
     (pin "1")
     (pin "2")
@@
       (effects (font (size 1.27 1.27)) hide)
     )
+    (property "Supplier" "Digi-Key" (at 87.63 90.17 0)
+      (effects (font (size 1.27 1.27)) hide)
+    )
+    (property "LibRef" "" (at 87.63 90.17 0)
+      (effects (font (size 1.27 1.27)) hide)
+    )

Commit message: Fill in all part numbers, add pcbinv bom job
Parts:
- FB4: LibRef (none) -> 742792121
- R11, R12: LibRef (none) -> RC1206FR-075K1L; SKU (none) -> 311-5.10KFRCT-ND
- U9: value LD1117S33TR_SOT223 -> LD1117S33TR; SKU (none) -> 497-1242-1-ND
Changed lines of the file:
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@@
+      (effects (font (size 1.27 1.27)) hide)
+    )
+    (property "Description" "CAP CER 2.2uF 50V X7R 1206" (at 125.73 78.74 0)
       (effects (font (size 1.27 1.27)) hide)
     )
@@
       (effects (font (size 1.27 1.27)) hide)
     )
-    (property "LibRef" "" (at 111.76 82.55 0)
+    (property "LibRef" "RC1206FR-075K1L" (at 111.76 82.55 0)
+      (effects (font (size 1.27 1.27)) hide)
+    )
+    (property "Description" "RES 5.1k Ohm 1% 1/4W 1206" (at 111.76 82.55 0)
+      (effects (font (size 1.27 1.27)) hide)
+    )
+    (property "SKU" "311-5.10KFRCT-ND" (at 111.76 82.55 0)
       (effects (font (size 1.27 1.27)) hide)
     )
@@
     )
     (property "SKU" "1276-1291-1-ND" (at 143.51 78.74 0)
+      (effects (font (size 1.27 1.27)) hide)
+    )
+    (property "Description" "CAP CER 2.2uF 50V X7R 1206" (at 143.51 78.74 0)
       (effects (font (size 1.27 1.27)) hide)
     )
@@
       (effects (font (size 1.27 1.27)) hide)
     )
-    (property "LibRef" "" (at 111.76 80.01 0)
+    (property "LibRef" "RC1206FR-075K1L" (at 111.76 80.01 0)
+      (effects (font (size 1.27 1.27)) hide)
+    )
+    (property "Description" "RES 5.1k Ohm 1% 1/4W 1206" (at 111.76 80.01 0)
+      (effects (font (size 1.27 1.27)) hide)
+    )
+    (property "SKU" "311-5.10KFRCT-ND" (at 111.76 80.01 0)
       (effects (font (size 1.27 1.27)) hide)
     )
@@
       (effects (font (size 1.27 1.27)))
     )
-    (property "Value" "LD1117S33TR_SOT223" (at 177.8 71.12 0)
+    (property "Value" "LD1117S33TR" (at 177.8 71.12 0)
       (effects (font (size 1.27 1.27)))
     )
@@
     )
     (property "LibRef" "" (at 177.8 74.93 0)
+      (effects (font (size 1.27 1.27)) hide)
+    )
+    (property "SKU" "497-1242-1-ND" (at 177.8 74.93 0)
       (effects (font (size 1.27 1.27)) hide)
     )
@@
       (effects (font (size 1.27 1.27)) hide)
     )
-    (property "LibRef" "" (at 135.89 74.93 0)
-      (effects (font (size 1.27 1.27)) hide)
-    )
+    (property "LibRef" "742792121" (at 135.89 74.93 0)
+      (effects (font (size 1.27 1.27)) hide)
+    )
+    (property "Description" "FERRITE BEAD 300 OHM 1206 1LN" (at 135.89 74.93 0)
+      (effects (font (size 1.27 1.27)) hide)
+    )

Commit message: Update to KiCAD 8, start adding CAN transceiver
Parts:
- renumbered C13 to C12, C12 to C13, C12 to C16, C12 to C17, FB4 to FB3, J1 to J3, U3 to U8

Commit message: ERC passing!
Parts:
- J3: symbol Connector:USB_C_Receptacle_USB2.0 -> Connector:USB_C_Receptacle_USB2.0_16P
Changed lines of the file:
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@@
 	)
 	(no_connect
-		(at 111.76 104.14)
+		(at 116.84 104.14)
 	)
 	(no_connect
@@
 	)
 	(no_connect
-		(at 132.08 104.14)
+		(at 127 104.14)
 	)
 	(no_connect
@@
 	)
 	(no_connect
-		(at 111.76 99.06)
+		(at 116.84 101.6)
 	)
 	(no_connect
@@
 	)
 	(no_connect
-		(at 132.08 99.06)
+		(at 127 101.6)
 	)
 	(wire
@@
 	(wire
 		(pts
-			(xy 121.92 74.93) (xy 121.92 91.44)
+			(xy 121.92 74.93) (xy 121.92 96.52)
 		)
 		(stroke
@@
 	(wire
 		(pts
-			(xy 121.92 111.76) (xy 121.92 116.84)
+			(xy 121.92 109.22) (xy 121.92 116.84)
 		)
 		(stroke
@@
 			)
 		)
-		(property "Description" "CAP CER 2.2uF 50V X7R 1206"
+		(property "Description" "Unpolarized capacitor, small symbol"
 			(at 125.73 78.74 0)
 			(effects
@@
 			)
 		)
-		(property "Description" ""
+		(property "Description" "Unpolarized capacitor, small symbol"
 			(at 193.04 78.74 0)
 			(effects
@@
 			)
 		)
-		(property "Description" ""
+		(property "Description" "Very low capacitance ESD protection diode, 2 data-line, SOT-23-6"
 			(at 121.92 101.6 0)
 			(effects
@@
 			)
 		)
-		(property "Description" "RES 5.1k Ohm 1% 1/4W 1206"
+		(property "Description" "Resistor, US symbol"
 			(at 111.76 82.55 0)
 			(effects
@@
 			)
 		)
-		(property "Description" ""
+		(property "Description" "Unpolarized capacitor, small symbol"
 			(at 161.29 78.74 0)
 			(effects
@@
 			)
 		)
-		(property "Description" "CAP CER 2.2uF 50V X7R 1206"
+		(property "Description" "Unpolarized capacitor, small symbol"
 			(at 143.51 78.74 0)
 			(effects
@@
 			)
 		)
-		(property "Description" "RES 5.1k Ohm 1% 1/4W 1206"
+		(property "Description" "Resistor, US symbol"
 			(at 111.76 80.01 0)
 			(effects
@@
 			)
 		)
-		(property "Description" ""
+		(property "Description" "800mA Fixed Low Drop Positive Voltage Regulator, Fixed Output 3.3V, SOT-223"
 			(at 177.8 74.93 0)
 			(effects
@@
 			)
 		)
-		(property "Description" "FERRITE BEAD 300 OHM 1206 1LN"
+		(property "Description" "Ferrite bead, small symbol"
 			(at 135.89 74.93 0)
 			(effects
@@
 	)
 	(symbol
-		(lib_id "Connector:USB_C_Receptacle_USB2.0")
+		(lib_id "Connector:USB_C_Receptacle_USB2.0_16P")
 		(at 87.63 90.17 0)
 		(unit 1)
@@
 			)
 		)
-		(property "Description" ""
+		(property "Description" "USB 2.0-only 16P Type-C Receptacle connector"
 			(at 87.63 90.17 0)
 			(effects

Commit message: Kate's suggestions, part 1
Parts:
- added R46, R47: 1, Resistor_SMD:R_1206_3216Metric, symbol Device:R_US
Connections:
- net +5V: now also C12.2
- net GND: now also R46.1, R47.1; no longer C12.1, C13.1
- net VBUS_IN: no longer C12.2
- new net: C12.1, R46.2
- new net: C13.1, R47.2
Other:
- moved on the sheet: C12, C13, C16, FB3

Commit message: Fix some BOM isues
Parts:
- R46, R47: LibRef P1.0RCT-ND -> ERJ-8RQF1R0V; SKU P120FCT-ND -> P1.0RCT-ND
Changed lines of the file:
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@@
 			)
 		)
-		(property "LibRef" "P1.0RCT-ND"
+		(property "LibRef" "ERJ-8RQF1R0V"
 			(at 143.51 88.9 0)
 			(effects
@@
 			)
 		)
-		(property "SKU" "P120FCT-ND"
+		(property "SKU" "P1.0RCT-ND"
 			(at 143.51 88.9 0)
 			(effects
@@
 			)
 		)
-		(property "LibRef" "P1.0RCT-ND"
-			(at 135.89 88.9 0)
-			(effects
-				(font
-					(size 1.27 1.27)
-				)
-				(hide yes)
-			)
-		)
-		(property "SKU" "P120FCT-ND"
-			(at 135.89 88.9 0)
-			(effects
+		(property "LibRef" "ERJ-8RQF1R0V"
+			(at 135.89 88.9 0)
+			(effects
+				(font
+					(size 1.27 1.27)
+				)
+				(hide yes)
+			)
+		)
+		(property "SKU" "P1.0RCT-ND"
+			(at 135.89 88.9 0)
+			(effects
