File: kicad_project/PowerUSBPort.kicad_sch (KiCad schematic)
At the start: 12 parts, among them J3 USB4105-GF-A, U8 USBLC6-2SC6, U9 LD1117S33TR

Commit message: Finish schematic and placement for all remaining RP2354 power passives
Changed lines of the file:
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@@
 		(pin "B9"
 		)
-		(pin "S1"
+		(pin "SH"
 		)
 		(instances
