File: kicad_project/MicroSDCard.kicad_sch (KiCad schematic)
At the start: 18 parts, among them J8 DM3AT, U14 74AHC1G04, U21 SN74AXC4T774, U22 AP22913W6-7

Commit message: Finish schematic and placement for all remaining RP2354 power passives
Connections:
- net GND: now also J8.SH (SHIELD); no longer J8.11 (SHIELD)
Changed lines of the file:
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@@
 		(pin "10"
 		)
-		(pin "11"
+		(pin "SH"
 		)
 		(pin "2"
